Commit message: slide sphere

File: catkin_ws/src/simple2wheeler/urdf/simple2wheeler.xacro (robot description, xacro)
@@ -7,4 +7,6 @@
         <material>Gazebo/Orange</material>
     </gazebo>
+<!--
+-->
     <gazebo>
         <plugin filename="libgazebo_ros_diff_drive.so" name="differential_drive_controller">
@@ -12,6 +14,6 @@
             <alwaysOn>true</alwaysOn>
             <updateRate>20</updateRate>
+            <rightJoint>joint_right_wheel</rightJoint>
             <leftJoint>joint_left_wheel</leftJoint>
-            <rightJoint>joint_right_wheel</rightJoint>
             <wheelSeparation>0.2</wheelSeparation>
             <wheelDiameter>0.2</wheelDiameter>
@@ -42,4 +44,26 @@
             </geometry>
             <material name="blue"/>
+        </visual>
+        <collision name="caster_front_collision">
+            <origin rpy="0 0 0" xyz="0.35 0 -0.05"/>
+            <geometry>
+                <sphere radius="0.05"/>
+            </geometry>
+            <surface>
+                <friction>
+                    <ode>
+                        <mu>0</mu>
+                        <mu2>0</mu2>
+                        <slip1>1.0</slip1>
+                        <slip2>1.0</slip2>
+                    </ode>
+                </friction>
+            </surface>
+        </collision>
+        <visual name="caster_front_visual">
+            <origin rpy="0 0 0" xyz="0.2 0 -0.05"/>
+            <geometry>
+                <sphere radius="0.05"/>
+            </geometry>
         </visual>
     </link>

Commit message: ohjausta parannettu vaihtamalla joint xyz +/- kulkijaan asennettu isommat renkaat

File: catkin_ws/src/simple2wheeler/urdf/simple2wheeler.xacro (robot description, xacro)
@@ -7,6 +7,4 @@
         <material>Gazebo/Orange</material>
     </gazebo>
-<!--
--->
     <gazebo>
         <plugin filename="libgazebo_ros_diff_drive.so" name="differential_drive_controller">
@@ -77,5 +75,5 @@
             <origin rpy="0 1.5707 1.5707" xyz="0 0 0"/>
             <geometry>
-                <cylinder length="0.04" radius="0.1"/>
+                <cylinder length="0.04" radius="0.15"/>
             </geometry>
         </collision>
@@ -83,5 +81,5 @@
             <origin rpy="0 1.5707 1.5707" xyz="0 0 0"/>
             <geometry>
-                <cylinder length="0.04" radius="0.1"/>
+                <cylinder length="0.04" radius="0.15"/>
             </geometry>
             <material name="blue"/>
@@ -89,5 +87,5 @@
     </link>
     <joint name="joint_right_wheel" type="continuous">
-        <origin rpy="0 0 0" xyz="-0.05 0.15 0 "/>
+        <origin rpy="0 0 0" xyz="-0.05 -0.15 0 "/>
         <child link="link_right_wheel"/>
         <parent link="link_chassis"/>
@@ -105,5 +103,5 @@
             <origin rpy="0 1.5707 1.5707" xyz="0 0 0"/>
             <geometry>
-                <cylinder length="0.04" radius="0.1"/>
+                <cylinder length="0.04" radius="0.15"/>
             </geometry>
         </collision>
@@ -111,11 +109,11 @@
             <origin rpy="0 1.5707 1.5707" xyz="0 0 0"/>
             <geometry>
-                <cylinder length="0.04" radius="0.1"/>
+                <cylinder length="0.04" radius="0.15"/>
             </geometry>
             <material name="blue"/>
         </visual>
     </link>
-    <joint name="joint_left_wheel" type="continuous">
-        <origin rpy="0 0 0" xyz="-0.05 -0.15 0 "/>
+     <joint name="joint_left_wheel" type="continuous">
+        <origin rpy="0 0 0" xyz="-0.05 0.15 0 "/>
         <child link="link_left_wheel"/>
         <parent link="link_chassis"/>
